Commit message: feat: v5-Finger über PhysX Mimic Joints, Servo-Aktuatormodell, Self-Collision
Ersetzt die Sehnendynamik-Kopplung per Script Node (1d0cd9c, ADR-009) — Branch dafür
auf 0fdbc62 zurückgesetzt, alter Stand als Tag backup/sehnendynamik-1d0cd9c, die
Experimente der Vorsession (Kraft-Rückwirkung, Mimic-Vorprüfungen) liegen in stash@{0}.

Mimic Joints (Stufe 1, linear): PIP←MCP, DIP←PIP, Daumen-IP←MCP, beide Hände
(18 Gelenke), gearing=-1/offset=0, hart (Isaac Sim 5.1 hat keine Mimic-Compliance).
Konfiguration zentral in setup_stage.py (MIMIC_JOINTS, configure_mimic_joints(),
von start.py jede Session gesetzt); configure_drives() lässt die Folgegelenke passiv.

Servo-Aktuatormodell nach NVIDIA Articulation Stability Guide / Robotiq-Tuning-Rezept
für MCP, Handgelenk, Unterarm, Daumen-Rotator (ST3215, 12 V): maxForce 2.94 Nm,
maxJointVelocity 270 °/s, Stiffness = maxForce / 5° (0.588 Nm/°), kritische
Dämpfung, Armature 5e-3 (Annahme). Folgegelenke: Armature 5e-4, 500 °/s. Vorher
500 Nm/° bei 2.94 Nm Kappung — der Antrieb sättigte bei 0.006° Fehler und wirkte
wie ein Relais. Experiment-Schalter in setup_stage.py dokumentieren die Varianten.
Arm/Kopf (3000-5000 Nm/°, maxForce inf) noch nicht umgestellt.

pib_upperbody_v5.usd: Action Graph auf OnPhysicsStep umgestellt (Graph-Prim
evaluationMode=Standalone, pipelineStage=pipelineStageOnDemand), Self-Collision am
root_joint wieder an (damit kein Wegfliegen/Schwingen mehr beim Tischkontakt),
Unterarm-Masse korrigiert (Override 30 g → autocomputed 0.229 kg, Trägheit
skaliert, gegen Onshape verifiziert) — URDFs ebenso.

v5-Gelenklimits korrigiert (upper_arm_left [-90°,90°], wrist_* [-90°,30°]),
config/pib_hand_config_v5.py neu.

Neue Werkzeuge:
- test_client_mimic_v5 — Kopplung ohne Last (nur MCP kommandiert)
- test_client_mimic_load_v5 — Finger gegen Tisch, Diagnose für Kopplung,
  Gelenkbereich, Chattern, MCP-Grenzen, NaN, Arm-Drift
- isaac_sim/tools/audit_asset.py — Asset-Inspektion: Massen USD/PhysX/URDF,
  Collider, Antriebe, effektive Gelenkträgheit, ω_n·Δt/ζ nach NVIDIA

Verifiziert: alle 10 MCPs frei (Δ ≤ 0.2°), index_left und alle vier linken Finger
gegen den Tisch — stabiler Stall bzw. Handgelenk gibt realistisch nach, Kopplung
≤ 0.1°, kein Ausbrechen.

Docs (Handoff, Sprint, ADR-010/011, CLAUDE.md) noch nicht nachgezogen.

Co-Authored-By: Claude Opus 5.5 <noreply@anthropic.com>

File: pib_upperbody_urdf_v5/robot.urdf (robot description, URDF)
Before this commit: robot pib_upperbody_urdf_v5, 47 links, 46 joints
Links:
- link urdf_forearm_left: mass 0.03 -> 0.229
- link urdf_forearm_right: mass 0.03 -> 0.229

File: ros2_ws/src/pib_description_v5/urdf/pib_upperbody_v5.urdf (robot description, URDF)
Before this commit: robot pib_upperbody_v5, 47 links, 46 joints
Links:
- link urdf_forearm_left: mass 0.03 -> 0.229
- link urdf_forearm_right: mass 0.03 -> 0.229
