Commit message: feat: Handgelenk-Pleuel modelliert, Grenzen v5-Handgelenk auf [-60°, 0°]
Das Handgelenk wird über ein Pleuel vom ST3215 angetrieben (Kurbel 6 mm, Pleuel
115 mm, Hebel 12 mm, Gestell 115,43 mm). Der Hebel schwenkt zwischen den Totlagen
nur 60° -> Grenzen [-60°, 0°] (in Onshape korrigiert, URDFs/setup_stage nachgezogen,
ohne Neuimport). Vorzeichen-Ausnahme: -60° = gebeugt (conventions.md).

config/pib_hand_config_v5.py: WRIST_LINKAGE, wrist_transmission() (analytisch),
wrist_lookup_table() für Isaac Labs RemotizedPDActuatorCfg (NVIDIA-Muster Spot-Knie,
gekappt bei 12 Nm), TRANSMISSIONS -> servo_actuator() rechnet Moment/Geschwindigkeit/
Armature aufs Gelenk um (Handgelenk Mitte: 5,87 Nm, 135 °/s, Armature x4).
USDs: Hand per bake_hand_asset_v5.py, Vollroboter per start.py aktualisiert.

Co-Authored-By: Claude Opus 5.5 <noreply@anthropic.com>

File: pib_hand_left_urdf_v5/robot.urdf (robot description, URDF)
Before this commit: robot pib_hand_left_v5, 18 links, 17 joints
Joints:
- joint wrist_left: limit lower=-1.5708 upper=0.523599 effort=10 velocity=10 -> lower=-1.0472 upper=0 effort=10 velocity=10

File: pib_upperbody_urdf_v5/robot.urdf (robot description, URDF)
Before this commit: robot pib_upperbody_urdf_v5, 47 links, 46 joints
Joints:
- joint wrist_left: limit lower=-1.5708 upper=0.523599 effort=10 velocity=10 -> lower=-1.0472 upper=0 effort=10 velocity=10
- joint wrist_right: limit lower=-1.5708 upper=0.523599 effort=10 velocity=10 -> lower=-1.0472 upper=0 effort=10 velocity=10

File: ros2_ws/src/pib_description_v5/urdf/pib_upperbody_v5.urdf (robot description, URDF)
Before this commit: robot pib_upperbody_v5, 47 links, 46 joints
Joints:
- joint wrist_left: limit lower=-1.5708 upper=0.523599 effort=10 velocity=10 -> lower=-1.0472 upper=0 effort=10 velocity=10
- joint wrist_right: limit lower=-1.5708 upper=0.523599 effort=10 velocity=10 -> lower=-1.0472 upper=0 effort=10 velocity=10
